File: pcb/pcb.kicad_pcb (KiCad board)
At the start: 2 copper layers, 136 x 91.7 mm, 56 parts, among them J1 BATT, J2 BATT, SW1 SW_SPST, SW10 SW_SPST, SW11 SW_SPST, SW12 SW_SPST, SW13 SW_SPST, SW14 SW_SPST, SW15 SW_SPST, SW16 SW_SPST, SW17 SW_SPST, SW18 SW_SPST, SW19 SW_SPST, SW2 SW_SPST, SW20 SW_SPST, SW21 SW_SPST, SW3 SW_SPST, SW4 SW_SPST, SW5 SW_SPST, SW6 SW_SPST, SW7 SW_SPST, SW8 SW_SPST, SW9 SW_SPST, U1 XIAO_nRF52840

Commit message: backup
Parts:
- removed J1: BATT, one:Battery
- removed J2: BATT, one:JST_SH_Battery_DUAL
- removed U1: XIAO_nRF52840, one:XIAO_nRF52840_DUAL
- added C1: 4u7, Capacitor_SMD:C_0402_1005Metric, F.Cu at (199.0, 78.1)
- added C10: 4u7, Capacitor_SMD:C_0402_1005Metric, F.Cu at (199.3, 66.8)
- added C11: 4u7, Capacitor_SMD:C_0402_1005Metric, F.Cu at (200.9, 82.5)
- added C12: 12p, Capacitor_SMD:C_0402_1005Metric, F.Cu at (133.2, 125.3)
- added C13: 12p, Capacitor_SMD:C_0402_1005Metric, F.Cu at (133.2, 124.3)
- added C2: 4u7, Capacitor_SMD:C_0402_1005Metric, F.Cu at (200.0, 78.1)
- added C3: 1u, Capacitor_SMD:C_0402_1005Metric, F.Cu at (201.0, 78.1)
- added C4: 4u7, Capacitor_SMD:C_0402_1005Metric, F.Cu at (194.5, 83.2)
- added C5: 1u, Capacitor_SMD:C_0402_1005Metric, F.Cu at (194.5, 82.2)
- added C6: 100n, Capacitor_SMD:C_0402_1005Metric, F.Cu at (202.5, 77.9)
- added C7: 4u7, Capacitor_SMD:C_0402_1005Metric, F.Cu at (193.9, 80.6)
- added C8: 1u, Capacitor_SMD:C_0402_1005Metric, F.Cu at (194.9, 80.5)
- added C9: 1u, Capacitor_SMD:C_0402_1005Metric, F.Cu at (132.3, 118.2)
- added F1: 500mA, Fuse:Fuse_0603_1608Metric, F.Cu at (199.1, 64.7)
- added J3: TYPE-C-31-M-12, PCM_marbastlib-various:USB_C_Receptacle_HRO_TYPE-C-31-M-12, F.Cu at (195.3, 57.9)
- added J4: 78171-0002, PCM_marbastlib-various:Molex_Pico-EZmate_78171-0002_1x02-1MP_P1.20mm_Vertical, F.Cu at (204.9, 81.1)
- added J5: TC2030_SWD, PCM_marbastlib-various:CON_TC2030_outlined, F.Cu at (139.4, 125.1)
- added L1: BLM15PX121SN1D, Inductor_SMD:L_0402_1005Metric, F.Cu at (197.8, 66.1)
- added L2: 10 uH, Inductor_SMD:L_0603_1608Metric, F.Cu at (131.0, 117.7)
- added R1: 5k1, Resistor_SMD:R_0402_1005Metric, F.Cu at (192.6, 64.2)
- added R2: 5k1, Resistor_SMD:R_0402_1005Metric, F.Cu at (197.8, 64.2)
- added R3: 10k, Resistor_SMD:R_0402_1005Metric, F.Cu at (195.9, 78.1)
- added R4: 47k, Resistor_SMD:R_0402_1005Metric, F.Cu at (197.9, 78.1)
- added R5: 1k5, Resistor_SMD:R_0402_1005Metric, F.Cu at (200.4, 81.0)
- added R6: 2k2, Resistor_SMD:R_0402_1005Metric, F.Cu at (196.9, 78.1)
- added R7: 10k, Resistor_SMD:R_0402_1005Metric, F.Cu at (131.3, 122.9)
- added R8: 10k, Resistor_SMD:R_0402_1005Metric, F.Cu at (131.1, 121.4)
- added SW22: RST, PCM_marbastlib-various:SW_T1A2QR, F.Cu at (134.8, 127.5)
- added U2: MAX17048, custom:DFN-8-1EP_2x2mm_P0.5mm_EP0.7x1.3mm, F.Cu at (202.8, 75.7)
- added U3: BQ24075, Package_DFN_QFN:VQFN-16-1EP_3x3mm_P0.5mm_EP1.6x1.6mm, F.Cu at (197.7, 81.3)
- added U4: SRV05-4, PCM_marbastlib-various:SOT-23-6-routable, F.Cu at (195.2, 65.2)
- added U5: nRF52840_E73-2G4M08S1C, PCM_marbastlib-various:nRF52840_E73-2G4M08S1C, F.Cu at (120.7, 120.9)
- added Y1: 32.768 KHz, Crystal:Crystal_SMD_2012-2Pin_2.0x1.2mm, F.Cu at (131.3, 124.8)
- moved G*** 82.5 mm to (222.2, 113.2) (x2)
- moved PWR1 5.61 mm to (206.1, 56.1)
Routing:
- net C0: track 186.0 -> 0.00 mm, vias 5 -> 0
- net R2: track 175.6 -> 0.00 mm, vias 16 -> 0
- net R0: track 165.5 -> 0.00 mm, vias 18 -> 0
- net C1: track 164.4 -> 0.00 mm, vias 5 -> 0
- net R1: track 161.3 -> 0.00 mm, vias 15 -> 0
- net C3: track 160.6 -> 0.00 mm, vias 8 -> 0
- net C2: track 145.9 -> 0.00 mm, vias 5 -> 0
- net C4: track 144.3 -> 0.00 mm, vias 8 -> 0
- net R3: track 134.9 -> 0.00 mm, vias 10 -> 0
- net C5: track 120.0 -> 0.00 mm, vias 7 -> 0
- net D+: track 0.00 -> 103.5 mm
- net D-: track 0.00 -> 101.9 mm
- net Net-(J1-Pin_1): track 48.5 -> 0.00 mm, vias 5 -> 0
- net B-: track 48.2 -> 0.00 mm, vias 4 -> 0
- net Net-(D21-A): track 28.2 -> 0.00 mm, vias 3 -> 0
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- removed copper zone on B.Cu, net (none)
- removed copper zone on F.Cu, net (none)
Other:
- outline, holes or cut-outs redrawn
- board text removed: "Ergonaut One v1.2 by yumagulovrn"
