File: pcb/pcb.kicad_sch (KiCad schematic)
At the start: 53 parts, among them J1 BATT, J2 BATT, SW1 SW_SPST, SW10 SW_SPST, SW11 SW_SPST, SW12 SW_SPST, SW13 SW_SPST, SW14 SW_SPST, SW15 SW_SPST, SW16 SW_SPST, SW17 SW_SPST, SW18 SW_SPST, SW19 SW_SPST, SW2 SW_SPST, SW20 SW_SPST, SW21 SW_SPST, SW3 SW_SPST, SW4 SW_SPST, SW5 SW_SPST, SW6 SW_SPST, SW7 SW_SPST, SW8 SW_SPST, SW9 SW_SPST, U1 XIAO_nRF52840

Commit message: backup
Parts:
- removed J1: BATT, one:Battery, symbol Connector:Conn_01x02_Pin
- removed J2: BATT, one:JST_SH_Battery_DUAL, symbol Connector:Conn_01x02_Pin
- removed PWR1: SW_SPDT, one:MSK-12C02_DUAL, symbol Switch:SW_SPDT
- removed U1: XIAO_nRF52840, one:XIAO_nRF52840_DUAL, symbol one:XIAO_nRF52840
- added C1, C10, C11, C2, C4, C7: 4u7, Capacitor_SMD:C_0402_1005Metric, symbol Device:C_Small
- added C12, C13: 12p, Capacitor_SMD:C_0402_1005Metric, symbol Device:C_Small
- added C3, C5, C8, C9: 1u, Capacitor_SMD:C_0402_1005Metric, symbol Device:C_Small
- added C6: 100n, Capacitor_SMD:C_0402_1005Metric, symbol Device:C_Small
- added F1: 500mA, Fuse:Fuse_0603_1608Metric, symbol Device:Polyfuse_Small
- added J3: TYPE-C-31-M-12, PCM_marbastlib-various:USB_C_Receptacle_HRO_TYPE-C-31-M-12, symbol Connector:USB_C_Receptacle_USB2.0
- added J4: 78171-0002, PCM_marbastlib-various:Molex_Pico-EZmate_78171-0002_1x02-1MP_P1.20mm_Vertical, symbol Connector_Generic_MountingPin:Conn_01x02_MountingPin
- added J5: TC2030_SWD, PCM_marbastlib-various:CON_TC2030_outlined, symbol PCM_marbastlib-various:TC2030_SWD
- added L1: BLM15PX121SN1D, Inductor_SMD:L_0402_1005Metric, symbol Device:L_Small
- added L2: 10 uH, Inductor_SMD:L_0603_1608Metric, symbol Device:L_Small
- added R1, R2: 5k1, Resistor_SMD:R_0402_1005Metric, symbol Device:R_Small
- added R3, R7, R8: 10k, Resistor_SMD:R_0402_1005Metric, symbol Device:R_Small
- added R4: 47k, Resistor_SMD:R_0402_1005Metric, symbol Device:R_Small
- added R5: 1k5, Resistor_SMD:R_0402_1005Metric, symbol Device:R_Small
- added R6: 2k2, Resistor_SMD:R_0402_1005Metric, symbol Device:R_Small
- added SW22: RST, PCM_marbastlib-various:SW_T1A2QR, symbol Switch:SW_Push
- added U2: MAX17048, custom:DFN-8-1EP_2x2mm_P0.5mm_EP0.7x1.3mm, symbol marbastlib-various:MAX17048
- added U3: BQ24075, Package_DFN_QFN:VQFN-16-1EP_3x3mm_P0.5mm_EP1.6x1.6mm, symbol Battery_Management:BQ24075RGT
- added U4: SRV05-4, PCM_marbastlib-various:SOT-23-6-routable, symbol PCM_marbastlib-various:SRV05-4
- added U5: nRF52840_E73-2G4M08S1C, PCM_marbastlib-various:nRF52840_E73-2G4M08S1C, symbol PCM_marbastlib-various:nRF52840_E73-2G4M08S1C
- added Y1: 32.768 KHz, Crystal:Crystal_SMD_2012-2Pin_2.0x1.2mm, symbol Device:Crystal_Small
Connections:
- net +5V: now also C1.1, C10.1, C2.1, C3.1, L1.2, U3.13 (IN), U5.27 (VBUS)
- net C0: now also U5.41 (P0.09/NFC1)
- net C1: now also U5.34 (P0.22)
- net C2: now also U5.43 (P0.10/NFC2)
- net C3: now also U5.28 (P0.15)
- net C4: now also U5.32 (P0.20)
- net C5: now also U5.33 (P0.13)
- net GND: now also C1.2, C10.2, C11.2, C12.2, C13.2, C2.2, C3.2, C4.2, C5.2, C6.2, C7.2, C8.2, C9.2, J3.A1 (GND), J3.A12 (GND), J3.B1 (GND), J3.B12 (GND), J3.S1 (SHIELD), J4.2 (Pin_2), J5.5 (GND), R1.2, R2.2, R3.2, R4.2, R5.2, R6.2, SW22.2, U2.1 (CTG), U2.4 (GND), U2.6 (QSTRT), U2.9 (GND), U3.15 (SYSOFF), U3.17 (VSS), U3.4 (~{CE}), U3.5 (EN2), U3.8 (VSS), U4.2 (VN), U5.21 (GND), U5.24 (GND), U5.5 (GND)
- net R0: now also U5.12 (P0.26)
- net R1: now also U5.14 (P0.06)
- net R2: now also U5.16 (P0.08)
- net R3: now also U5.30 (P0.17)
- new net: J3.B5 (CC2), R1.1
- new net: C13.1, U5.13 (P0.01/XL2), Y1.1
- new net: C12.1, U5.11 (P0.00/XL1), Y1.2
- new net: R6.1, U3.16 (ISET)
- new net: R3.1, U3.1 (TS)
- new net: J3.A5 (CC1), R2.1
- new net: F1.1, L1.1
- new net +BATT: C6.1, C7.1, C8.1, J4.1 (Pin_1), U2.2 (CELL), U2.3 (VDD), U3.2 (BAT), U3.3 (BAT)
- new net +VSW: C11.1, C4.1, C5.1, U3.10 (OUT), U3.11 (OUT), U3.6 (EN1), U5.23 (VDDH)
- new net ALERT: U2.5 (~{ALRT})
- new net D+: J3.A6 (D+), J3.B6 (D+), U4.1 (IO1), U5.31 (D+)
- new net D-: J3.A7 (D-), J3.B7 (D-), U4.6 (IO4), U5.29 (D-)
- new net DCCH: L2.1, U5.25 (DCCH)
- new net ILIM: R5.1, U3.12 (ILIM)
- new net LED_B: U5.38 (P1.02)
- new net LED_G: U5.36 (P1.00)
- new net RST: J5.3 (~{RST}), SW22.1, U5.26 (P0.18/~{RESET})
- new net SCL: R8.2, U2.7 (SCL), U5.17 (P1.09)
- new net SDA: R7.2, U2.8 (SDA), U5.15 (P0.05/AIN3)
- new net SWDCLK: J5.4 (SWCLK), U5.39 (SWDCLK)
- new net SWDIO: J5.2 (SWDIO), U5.37 (SWDIO)
- new net TMR: R4.1, U3.14 (TMR)
- new net VBUS: F1.2, J3.A4 (VBUS), J3.A9 (VBUS), J3.B4 (VBUS), J3.B9 (VBUS), U4.5 (VP)
- new net VDD: C9.1, J5.1 (VCC), L2.2, R7.1, R8.1, U5.19 (VDD)
- new net wk: U5.22 (P0.07)
- new net ~{CHG}: U3.9 (~{CHG})
- no-connect marks 8 -> 14
Other:
- note added: "Battery management"
- note added: "ESD input protection"
- note added: "External DCCH inductor for DC-DC HV input mode"
- note added: "External LF crystal for lower idle power"
- note added: "Fuel Gauge"
- note added: "Programming header"
- note added: "Pull-ups for i2c"
- note added: "TMR: (10 x 48 s/kOhm) * 47 kOhm = 22560s = 6.27h ILIM: 1550 AOhm / 1500 Ohm = 1.03 A = 1030 mA ISET: 890 AOhm / 2200 Ohm = 0.404 A = 440 mA EN1: 1, EN2: 0 = 475 mA MAX TS: 10 kOhm to GND = no OTP"
- note added: "USB Port"
- note added: "nRF52 module with peripherals"
- moved on the sheet: D1, D10, D11, D12, D13, D14, D15, D16, D17, D18, D19, D2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
